File: wlan-thermostat.kicad_sch (KiCad schematic)
At the start: 0 parts

Commit message: Initial board version
Parts:
- added C1, C2: 1uF, Capacitor_SMD:C_0603_1608Metric_Pad1.08x0.95mm_HandSolder, symbol Device:C
- added C1: 10uF, Capacitor_SMD:C_0603_1608Metric_Pad1.08x0.95mm_HandSolder, symbol Device:C
- added F1: Fuse, Fuse:Fuse_1206_3216Metric_Pad1.42x1.75mm_HandSolder, symbol Device:Fuse
- added H1, H2: MountingHole, MountingHole:MountingHole_3.2mm_M3, symbol Mechanical:MountingHole
- added IC1: ME6211C33M5G-N, SOT95P270X145-5N, symbol Chof747 Voltage Regulators:ME6211C33M5G-N
- added J2, J3: Conn_01x02, Connector_PinHeader_2.54mm:PinHeader_1x02_P2.54mm_Vertical, symbol Connector_Generic:Conn_01x02
- added J3: PROG_HDR, Connector_PinHeader_2.54mm:PinHeader_1x06_P2.54mm_Vertical, symbol Connector_Generic:Conn_01x06
- added JP1: PWR_PROG, Connector_PinHeader_2.54mm:PinHeader_1x02_P2.54mm_Vertical, symbol Jumper:Jumper_2_Open
- added Q1, Q2: SS8050-G, Package_TO_SOT_SMD:SOT-23, symbol Device:Q_NPN_BCE
- added R10, R2, R3, R7, R8, R9: 10k, Resistor_SMD:R_0603_1608Metric_Pad0.98x0.95mm_HandSolder, symbol Device:R
- added R14, R15: 22k, Resistor_SMD:R_0603_1608Metric_Pad0.98x0.95mm_HandSolder, symbol Device:R
- added R16, R17: 1k, Resistor_SMD:R_0603_1608Metric_Pad0.98x0.95mm_HandSolder, symbol Device:R
- added SW1: SW_Push, Button_Switch_THT:SW_PUSH_6mm, symbol Switch:SW_Push
- added SW4: RotaryEncoder_Switch, PEC12R3120FS0012, symbol Chof747 Controls:PEC12R-3120F-S0012
- added U1: ESP-12F, RF_Module:ESP-12E, symbol RF_Module:ESP-12F
- added U2: SHT4x, Sensor_Humidity:Sensirion_DFN-4_1.5x1.5mm_P0.8mm_SHT4x_NoCentralPad, symbol Sensor_Humidity:SHT4x
- added U3: SSD1306, Chof747 Footprints:AZ Delivery SS1306 OLED, symbol Cho747 Displays:SSD1306
Connections:
- new net: Q2.1 (B), R3.2
- new net: R8.2, U1.3 (EN)
- new net: R14.1, R16.2, SW4.A1 (CHANNEL_A)
- new net: R15.1, R17.2, SW4.B1 (CHANNEL_B)
- new net: Q1.1 (B), R2.2
- new net +3V3: C1.1, C2.1, IC1.5 (VOUT), JP1.1 (A), R10.1, R14.2, R15.2, R7.1, R8.1, R9.1, U1.8 (VCC), U2.3 (VDD), U3.2 (VCC)
- new net +5V: C1.1, IC1.1 (VIN), IC1.3 (CE), J2.1 (Pin_1)
- new net 3v3PROG: F1.2, J3.1 (Pin_1)
- new net 3v3PROG_SAVE: F1.1, JP1.2 (B)
- new net DTR: J3.6 (Pin_6), Q2.3 (E), R2.1
- new net GND: C1.2, C1.2, C2.2, IC1.2 (VSS), J2.2 (Pin_2), J3.2 (Pin_2), J3.2 (Pin_2), SW1.2, SW4.1 (COM), SW4.C1 (COMMON), U1.15 (GND), U2.4 (VSS), U3.1 (GND)
- new net GPIO12_RENDAT: R17.1, U1.6 (GPIO12)
- new net GPIO13_RENBTN: SW4.2 (NO), U1.7 (GPIO13)
- new net GPIO14_RENCLK: R16.1, U1.5 (GPIO14)
- new net GPIO15_RELAY: J3.1 (Pin_1), U1.16 (GPIO15)
- new net GPIO3_RX: J3.3 (Pin_3), U1.21 (GPIO3/RXD)
- new net GPIO4_SDA: R10.2, U1.19 (GPIO4), U2.1 (SDA), U3.4 (SDA)
- new net GPIO4_TX: J3.4 (Pin_4), U1.22 (GPIO1/TXD)
- new net GPIO5_SCL: R9.2, U1.20 (GPIO5), U2.2 (SCL), U3.3 (SCL)
- new net RTS: J3.5 (Pin_5), Q1.3 (E), R3.1
- new net ~{GPIO0}: Q2.2 (C), U1.18 (GPIO0)
- new net ~{RESET}: Q1.2 (C), R7.2, SW1.1, U1.1 (~{RST})
- no-connect marks 0 -> 11
Other:
- note added: "OLED Display"
- note added: "Power Connection"
- note added: "Programming & Auto-Reset"
- note added: "Programming Header"
- note added: "Relay Connector"
- note added: "Reset Button"
- note added: "Rotary Encoder"
- note added: "Temperature & Humidity Sensor"
- note added: "Voltage Regulation"
- title: (none) -> Thermostate Front Module
