File: front-panel/wlan-thermo-front-panel.kicad_pcb (KiCad board)
At the start: 2 copper layers, 54.7 x 43.5 mm, 26 parts, among them IC1 ME6211C33M5G-N, J1 PROG_HDR, J2 Conn_01x02, J3 Conn_01x02, Q1 UMH3N, SW1 SW_Push, SW2 RotaryEncoder_Switch, U1 ESP-12F, U2 SHT4x, U3 SSD1306

Commit message: external version of temp sensor
Parts:
- added J4: SHT4x Out, Chof747 Footprints:JUSHUO-AFC10-S04QCA 1x4 Horizontal (JST SH), F.Cu at (144.9, 42.0)
- added J5: pwr-t, Chof747 Footprints:Solder Pad 1x2 1.5x3, F.Cu at (160.0, 70.3)
- added J6: i2c-t, Chof747 Footprints:Solder Pad 1x2 1.5x3, B.Cu at (160.0, 70.3)
- added REF**: Mousebites, Chof747 Board Modifications:Mousebites, F.Cu at (152.0, 70.3)
- J3: value Conn_01x02 -> Relay
- moved U2 31.5 mm to (155.8, 70.3), turned to -90 degrees
- moved R4 1.68 mm to (138.8, 49.3)
- moved R6 1.68 mm to (140.5, 49.3)
- moved R3 1.68 mm to (144.8, 49.3)
- moved R5 1.68 mm to (146.7, 49.3)
Connections:
- U2 pad 1: GPIO4_SDA -> Net-(J6-Pin_2)
- U2 pad 2: GPIO5_SCL -> Net-(J6-Pin_1)
- U2 pad 3: +3V3 -> Net-(J5-Pin_2)
- U2 pad 4: GND -> Net-(J5-Pin_1)
Routing:
- net GPIO5_SCL: track 62.3 -> 44.4 mm
- net +3V3: track 131.8 -> 117.0 mm, vias 4 -> 2
- net GND: track 51.6 -> 66.0 mm, vias 6 -> 7
- net GPIO4_SDA: track 58.1 -> 45.9 mm
- net Net-(J6-Pin_1): track 0.00 -> 6.34 mm, vias 0 -> 1
- net Net-(J5-Pin_2): track 0.00 -> 5.08 mm
- net Net-(J5-Pin_1): track 0.00 -> 4.76 mm
- net Net-(J6-Pin_2): track 0.00 -> 4.28 mm, vias 0 -> 1
- net Net-(SW2-CHANNEL_A): track 6.16 -> 4.49 mm
- net GPIO14_RENCLK: track 43.6 -> 42.1 mm
- net GPIO12_RENDAT: track 38.0 -> 36.6 mm
- net Net-(SW2-CHANNEL_B): track 6.13 -> 4.96 mm
Other:
- board size 54.7 x 43.5 mm -> 67.7 x 43.5 mm
