File: front-panel/wlan-thermo-front-panel.kicad_sch (KiCad schematic)
At the start: 25 parts, among them IC1 ME6211C33M5G-N, J2 Conn_01x02, J3 Conn_01x02, J3 PROG_HDR, Q1 UMH3N, SW1 SW_Push, SW4 RotaryEncoder_Switch, U1 ESP-12F, U2 SHT4x, U3 SSD1306

Commit message: crc checked first version of board with backend shelly
Parts:
- removed C1, C2: 1uF, Capacitor_SMD:C_0603_1608Metric_Pad1.08x0.95mm_HandSolder, symbol Device:C
- removed H1, H2: MountingHole, MountingHole:MountingHole_3.2mm_M3, symbol Mechanical:MountingHole
- removed IC1: ME6211C33M5G-N, SOT95P270X145-5N, symbol Chof747 Voltage Regulators:ME6211C33M5G-N
- removed J2, J3: Conn_01x02, Connector_PinHeader_2.54mm:PinHeader_1x02_P2.54mm_Vertical, symbol Connector_Generic:Conn_01x02
- added J2: Device Connector, Connector_PinHeader_1.27mm:PinHeader_1x07_P1.27mm_Vertical, symbol Connector_Generic:Conn_01x07
- SW1: footprint Button_Switch_THT:SW_PUSH_6mm -> Chof747 Footprints:KEY-SMD_L3.9-W3.0-LS5.0-EH
Connections:
- net +3V3: now also J2.4 (Pin_4)
- net GND: now also J2.7 (Pin_7)
- net GPIO4_SDA: now also RN1.2; no longer RN1.4
- net GPIO5_SCL: now also RN1.1; no longer RN1.3
- net ~{GPIO0_RENBTN_FLASH}: now also RN1.3; no longer RN1.1
- net ~{RESET}: now also J2.5 (Pin_5)
- net GPIO13_RELAY renamed GPIO13_RX1
- net GPIO13_RX1: now also J2.3 (Pin_3)
- net GPIO2 renamed GPIO2_RELAY
- net GPIO2_RELAY: now also RN1.4, J2.6 (Pin_6); no longer RN1.2
- no-connect marks 10 -> 12
Other:
- note removed: "Power Connection"
- note removed: "Voltage Regulation"

Commit message: minor changes
Parts:
- added JP2: Wake enable, Jumper:SolderJumper-2_P1.3mm_Open_Pad1.0x1.5mm, symbol Jumper:SolderJumper_2_Open
Connections:
- net ~{RESET}: now also JP2.1 (A)
- net GPIO16_WAKE: now reaches U1.4 (GPIO16)
- net GPIO16_WAKE: now also JP2.2 (B)
- no-connect marks 12 -> 11
Changed lines of the file:
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@@
 	)
 	(no_connect
-		(at 67.31 68.58)
-	)
-	(no_connect
 		(at 48.26 163.83)
 	)
@@
 	(wire
 		(pts
+			(xy 156.21 128.27) (xy 162.56 128.27)
+		)
+		(stroke
+			(width 0)
+			(type default)
+		)
+	)
+	(wire
+		(pts
 			(xy 113.03 49.53) (xy 113.03 62.23)
 		)
@@
 	(wire
 		(pts
+			(xy 67.31 68.58) (xy 72.39 68.58)
+		)
+		(stroke
+			(width 0)
+			(type default)
+		)
+	)
+	(wire
+		(pts
 			(xy 67.31 58.42) (xy 72.39 58.42)
 		)
@@
 		)
 	)
+	(global_label "GPIO16_WAKE"
+		(shape input)
+		(at 72.39 68.58 0)
+		(fields_autoplaced yes)
+		(effects
+			(font
+				(size 1.27 1.27)
+			)
+			(justify left)
+		)
+		(property "Intersheetrefs" "${INTERSHEET_REFS}"
+			(at 88.1961 68.58 0)
+			(effects
+				(font
+					(size 1.27 1.27)
+				)
+				(justify left)
+				(hide yes)
+			)
+		)
+	)
 	(global_label "GPIO4_TX"
 		(shape output)
@@
 		)
 	)
+	(global_label "GPIO16_WAKE"
+		(shape input)
+		(at 170.18 128.27 0)
+		(fields_autoplaced yes)
+		(effects
+			(font
+				(size 1.27 1.27)
+			)
+			(justify left)
+		)
+		(property "Intersheetrefs" "${INTERSHEET_REFS}"
+			(at 185.9861 128.27 0)
+			(effects
+				(font
+					(size 1.27 1.27)
+				)
+				(justify left)
+				(hide yes)
+			)
+		)
+	)
 	(global_label "GPIO5_SCL"
 		(shape bidirectional)
@@
 					(unit 1)
 				)
+			)
+		)
+	)
+	(symbol
+		(lib_id "Jumper:SolderJumper_2_Open")
+		(at 166.37 128.27 0)
+		(unit 1)
+		(exclude_from_sim yes)
+		(in_bom no)
+		(on_board yes)
+		(dnp no)
+		(property "Reference" "JP2"
+			(at 166.624 131.064 0)
+			(effects
+				(font
+					(size 1.27 1.27)
+				)
+			)
+		)
+		(property "Value" "Wake enable"
+			(at 175.514 124.968 0)
+			(effects
+				(font
+					(size 1.27 1.27)
+				)
+			)
+		)
+		(property "Footprint" "Jumper:SolderJumper-2_P1.3mm_Open_Pad1.0x1.5mm"
+			(at 166.37 128.27 0)
+			(effects
+				(font
+					(size 1.27 1.27)
+				)
+				(hide yes)
+			)
+		)
+		(property "Datasheet" "~"
+			(at 166.37 128.27 0)
+			(effects
+				(font
+					(size 1.27 1.27)
+				)
+				(hide yes)
+			)
+		)
+		(property "Description" "Solder Jumper, 2-pole, open"
+			(at 166.37 128.27 0)
+			(effects
+				(font
+					(size 1.27 1.27)
+				)
+				(hide yes)
+			)
+		)
+		(pin "2"
+		)
+		(pin "1"
+		)
+		(instances
+			(project ""
+				(path "/e8426e51-e5a9-4642-8277-6d3f50e0e523"
+					(reference "JP2")
+					(unit 1)
+				)
